Commit message: Updated xacro files (to match kraken prefab)
Signed-off-by: Paweł Budziszewski <pawel.budziszewski@robotec.ai>

File: Project/Assets/robotec_freezed_urdf_chasis/kraken_chasis.xacro (robot description, xacro)
@@ -53,7 +53,7 @@
        </collision>
        <collision>
-        <origin rpy="1.570796 -0.000000 1.570796" xyz="2.565201 0.000000 0.432055"/>
-        <geometry>
-           <box size="0.513190 0.131902 0.055878"/>
+        <origin rpy="1.570796 -0.000000 1.570796" xyz="2.5402429 0.000000 0.562592"/>
+        <geometry>
+           <box size="0.437199 0.131902 0.055878"/>
          </geometry>
        </collision>
@@ -72,7 +72,26 @@
       </inertial>
       <visual>
-        <origin rpy="0 1.571 0" xyz="0 0 ${wheel_width}"/>
-        <geometry>
-          <mesh filename="meshes/Wheels/WheelRight.dae" scale="0.6 0.6 0.6"/>
+        <origin rpy="0 1.571 0" xyz="0 0 0"/>
+        <geometry>
+          <mesh filename="meshes/Wheels/WheelRight.dae" scale="1 1 1"/>
+        </geometry>
+      </visual>
+      <collision>
+        <origin rpy="0 0 0" xyz="0 0 ${-wheel_width/2}"/>
+        <geometry>
+          <cylinder radius="${wheel_radius}" length="${wheel_width}" />
+        </geometry>
+      </collision>
+    </link>
+    <link name="wheel_rear_left_link">
+      <inertial>
+        <origin rpy="0 0 0" xyz="0 0.0 ${wheel_width}"/>
+        <mass value="24.5"/>
+        <inertia ixx="0.787" ixy="0.0" ixz="0.0" iyy="0.787" iyz="0.0" izz="1.309"/>
+      </inertial>
+      <visual>
+        <origin rpy="0 1.571 0 " xyz="0 0 0.0"/>
+        <geometry>
+          <mesh filename="meshes/Wheels/WheelLeft.dae" scale="1 1 1"/>
         </geometry>
       </visual>
@@ -84,26 +103,7 @@
       </collision>
     </link>
-    <link name="wheel_rear_left_link">
-      <inertial>
-        <origin rpy="0 0 0" xyz="0 0.0 ${wheel_width}"/>
-        <mass value="24.5"/>
-        <inertia ixx="0.787" ixy="0.0" ixz="0.0" iyy="0.787" iyz="0.0" izz="1.309"/>
-      </inertial>
-      <visual>
-        <origin rpy="0 -1.571 0 " xyz="0 0 0.0"/>
-        <geometry>
-          <mesh filename="meshes/Wheels/WheelLeft.dae" scale="0.6 0.6 0.6"/>
-        </geometry>
-      </visual>
-      <collision>
-        <origin rpy="0 0 0" xyz="0 0 -${wheel_width/2}"/>
-        <geometry>
-          <cylinder radius="${wheel_radius}" length="${wheel_width}" />
-        </geometry>
-      </collision>
-    </link>
     <link name="wheel_front_right_link">
       <inertial>
-        <origin rpy="0 0 0" xyz="0 0.0 ${-wheel_width/2}"/>
+        <origin rpy="0 0 0" xyz="0 0.0 ${wheel_width/2}"/>
         <mass value="24.5"/>
         <inertia ixx="0.787" ixy="0.0" ixz="0.0" iyy="0.787" iyz="0.0" izz="1.309"/>
@@ -112,5 +112,5 @@
         <origin rpy="0 1.571 0" xyz="0 0 0"/>
         <geometry>
-          <mesh filename="meshes/Wheels/WheelRight.dae" scale="0.6 0.6 0.6"/>
+          <mesh filename="meshes/Wheels/WheelRight.dae" scale="1 1 1"/>
         </geometry>
       </visual>
@@ -129,7 +129,7 @@
       </inertial>
       <visual>
-        <origin rpy="0 -1.571 0" xyz="0 0 ${wheel_width}"/>
-        <geometry>
-          <mesh filename="meshes/Wheels/WheelLeft.dae" scale="0.6 0.6 0.6"/>
+        <origin rpy="0 1.571 0" xyz="0 0 0"/>
+        <geometry>
+          <mesh filename="meshes/Wheels/WheelLeft.dae" scale="1 1 1"/>
         </geometry>
       </visual>
@@ -144,5 +144,5 @@
       <inertial>
         <origin rpy="0 0 -1.571" xyz="0 0 -0.04"/>
-        <mass value="1"/>
+        <mass value="20.0"/>
         <inertia ixx="1" ixy="0.0" ixz="0.0" iyy="1" iyz="0.0" izz="1"/>
       </inertial>
@@ -157,5 +157,5 @@
       <inertial>
         <origin rpy="0 0 -1.571" xyz="0 0 -0.04"/>
-        <mass value="1"/>
+        <mass value="20.0"/>
         <inertia ixx="1" ixy="0.0" ixz="0.0" iyy="1" iyz="0.0" izz="1"/>
       </inertial>
@@ -168,12 +168,12 @@
     </link>
     <joint name="wheel_rear_right_joint" type="continuous">
+      <origin rpy="-1.570796 0.000000 0.000000" xyz="0.000000 ${-wheel_base_rear} ${wheel_radius}"/>
+      <parent link="base_link"/>
+      <child link="wheel_rear_right_link"/>
+      <axis xyz="0.0 0.0 1.0"/>
+      <limit effort="1000000.0" velocity="1000.0"/>
+    </joint>
+    <joint name="wheel_rear_left_joint" type="continuous">
       <origin rpy="-1.570796 -0.000000 0.000000" xyz="0.000000 ${wheel_base_rear} ${wheel_radius}"/>
-      <parent link="base_link"/>
-      <child link="wheel_rear_right_link"/>
-      <axis xyz="0.0 0.0 1.0"/>
-      <limit effort="1000000.0" velocity="1000.0"/>
-    </joint>
-    <joint name="wheel_rear_left_joint" type="continuous">
-      <origin rpy="-1.570796 -0.000000 0.000000" xyz="0.000000 ${-wheel_base_rear} ${wheel_radius}"/>
       <parent link="base_link"/>
       <child link="wheel_rear_left_link"/>
@@ -211,40 +211,3 @@
       <limit effort="1000000.0" lower="-0.5235" upper="0.5235" velocity="100"/>
     </joint>
-<!--
-    <link name="manipulator_link_0_old">
-      <inertial>
-        <origin rpy="0.1745 0 0" xyz="0.0 -0.6 2.0"/>
-        <mass value="25.0"/>
-        <inertia ixx="0.002" ixy="0.0" ixz="0.0" iyy="0.068" iyz="0.0" izz="0.067"/>
-      </inertial>
-      <visual>
-        <origin rpy="-0.174533 0 0" xyz="0.9 -0.65 2.4"/>
-        <geometry>
-          <box size = "0.1 0.1 2.0"/>
-        </geometry>
-      </visual>
-      <visual>
-        <origin rpy="-0.174533 0 0" xyz="-0.9 -0.65 2.4"/>
-        <geometry>
-          <box size = "0.1 0.1 2.0"/>
-        </geometry>
-      </visual>
-      <collision>
-        <origin rpy="-0.174533 0 0" xyz="0.9 -0.65 2.4"/>
-        <geometry>
-          <box size = "0.1 0.1 2.0"/>
-        </geometry>
-      </collision>
-        <collision>
-        <origin rpy="-0.174533 0 0" xyz="-0.9 -0.65 2.4"/>
-        <geometry>
-          <box size = "0.1 0.1 2.0"/>
-        </geometry>
-      </collision>
-    </link>
-    <joint name="manipulator_joint_0" type="fixed">
-      <origin rpy="0 0 0" xyz="${manip_x+0.003927} ${manip_y} ${manip_z-1.0}"/>
-      <parent link="base_link"/>
-      <child link="manipulator_link_0_old"/>
-    </joint>  -->
 </robot>

File: Project/Assets/robotec_freezed_urdf_chasis/kraken_manipulator.xacro (robot description, xacro)
@@ -8,5 +8,5 @@
         <origin rpy="0.1745 0 0" xyz="0.0 -0.6 2.0"/>
         <mass value="25.0"/>
-        <inertia ixx="0.002" ixy="0.0" ixz="0.0" iyy="0.068" iyz="0.0" izz="0.067"/>
+        <inertia ixx="1.0" ixy="0.0" ixz="0.0" iyy="1.0" iyz="0.0" izz="1.0"/>
       </inertial>
       <visual>
@@ -16,4 +16,5 @@
         </geometry>
       </visual>
+      <!--
       <collision>
         <origin rpy="1.570798 1.396264 4.712389" xyz="0.485927 -0.460373 1.404769"/>
@@ -28,6 +29,7 @@
          </geometry>
        </collision>
+       -->
        <collision>
-        <origin rpy="-0.174561 0.000000 0.000000" xyz="-0.646611 -0.254306 2.573430"/>
+        <origin rpy="-0.0872664626 0.000000 0.000000" xyz="-0.3812585 -0.374285 2.5734301"/>
         <geometry>
            <box size="2.087586 0.088237 0.062286"/>
@@ -42,5 +44,5 @@
       </inertial>
       <visual>
-        <origin rpy="0 0 -1.571" xyz="0.0 0.0 0"/>
+        <origin rpy="0 0 -1.571" xyz="0.2528269 0.0 0"/>
         <geometry>
           <mesh filename="meshes/VacuumMechanismPart01/VacuumMechanismPart01.dae" scale="1 1 1"/>
@@ -48,5 +50,5 @@
       </visual>
       <collision>
-        <origin rpy="-0.001888 -0.000000 0.000000" xyz="0.000000 0.062564 -0.000045"/>
+        <origin rpy="-0.000 -0.000000 0.000000" xyz="0.000000 0.062564 -0.000045"/>
         <geometry>
            <box size="2.019587 0.172379 0.067739"/>
@@ -57,6 +59,6 @@
       <inertial>
         <origin rpy="0 0 0" xyz="0.0 0.0 0.0"/>
-        <mass value="10.0"/>
-        <inertia ixx="0.05" ixy="0.0" ixz="0.0" iyy="0.05" iyz="0.0" izz="0.05"/>
+        <mass value="25.0"/>
+        <inertia ixx="0.804004" ixy="0.0" ixz="0.0" iyy="0.9002936" iyz="0.0" izz="1.0483408"/>
       </inertial>
       <visual>
@@ -66,4 +68,5 @@
         </geometry>
       </visual>
+      <!--
       <collision>
         <origin rpy="0.0 0.0 0.0" xyz="0.0 0.0 0.0"/>
@@ -72,4 +75,5 @@
          </geometry>
        </collision>
+       -->
        <collision>
         <origin rpy="-1.570829 0 0 " xyz="-0.066974 -0.2 -0.000000"/>
@@ -83,6 +87,6 @@
       <inertial>
         <origin rpy="0 0 0" xyz="0.0 0.0 0.0"/>
-        <mass value="5.0"/>
-        <inertia ixx="0.01" ixy="0.0" ixz="0.0" iyy="0.01" iyz="0.0" izz="0.01"/>
+        <mass value="10.0"/>
+        <inertia ixx="0.5" ixy="0.0" ixz="0.0" iyy="0.5" iyz="0.0" izz="0.2"/>
       </inertial>
       <visual>
@@ -92,4 +96,5 @@
         </geometry>
       </visual>
+      <!--
       <collision>
         <origin rpy="0 0 0" xyz="0 0 0.0"/>
@@ -104,4 +109,5 @@
          </geometry>
        </collision>
+      -->
     </link>
     <!-- Nozzle02 -->
@@ -109,9 +115,9 @@
       <inertial>
         <origin rpy="0 0 0" xyz="0.0 0.0 0.0"/>
-        <mass value="5.0"/>
-        <inertia ixx="0.01" ixy="0.0" ixz="0.0" iyy="0.01" iyz="0.0" izz="0.01"/>
+        <mass value="10.0"/>
+        <inertia ixx="0.5" ixy="0.0" ixz="0.0" iyy="0.5" iyz="0.0" izz="0.2"/>
       </inertial>
       <visual>
-        <origin rpy="0 -1.571 0" xyz="0.0 0.0 0"/>
+        <origin rpy="0 -1.4835298642 0" xyz="0.0 0.0 0"/>
         <geometry>
           <mesh filename="meshes/VacuumNozzle02/VacuumNozzle02.dae" scale="1 1 1"/>
@@ -132,5 +138,5 @@
     <!-- Joint that moves manipulator along Z-Axis -->
     <joint name="kraken_manipulator_joint_1" type="prismatic">
-      <origin rpy="-0.1745 0 0" xyz="${manip_x-0.650001} -0.511055 1.6569"/>
+      <origin rpy="-0.0872664626 0 0" xyz="${manip_x-0.650001} -0.511055 1.6569"/>
       <parent link="base_link"/>
       <child link="kraken_manipulator_link_1"/>
@@ -146,5 +152,5 @@
       <axis xyz="0.0 0.0 1.0"/>
       <dynamics damping="2.0" friction="1.0"/>
-      <limit effort="1000.0" lower="-1.0" upper="1.0" velocity="1.0"/>
+      <limit effort="1000.0" lower="-0.8" upper="1.2" velocity="1.0"/>
     </joint>
     <!-- Nozzle -->
@@ -155,5 +161,5 @@
       <axis xyz="0.0 0.0 1.0"/>
       <dynamics damping="2.0" friction="1.0"/>
-      <limit effort="1000.0" lower="0" upper="0.28" velocity="1.0"/>
+      <limit effort="1000.0" lower="0" upper="0.3" velocity="1.0"/>
     </joint>
     <!-- Nozzle02 -->
@@ -164,5 +170,5 @@
       <axis xyz="0.0 0.0 1.0"/>
       <dynamics damping="2.0" friction="1.0"/>
-      <limit effort="1000.0" lower="0" upper="0.28" velocity="1.0"/>
+      <limit effort="1000.0" lower="0" upper="0.3" velocity="1.0"/>
     </joint>
 </robot>

Commit message: Fixed manipulator stability and added auxiliary objects
Signed-off-by: Paweł Budziszewski <pawel.budziszewski@robotec.ai>

File: Project/Assets/robotec_freezed_urdf_chasis/kraken_chasis.xacro (robot description, xacro)
@@ -167,4 +167,11 @@
       </visual>
     </link>
+    <link name="lidar_mount">
+      <inertial>
+        <origin rpy="0 0 0" xyz="0 0 0"/>
+        <mass value="1.0"/>
+        <inertia ixx="0.1" ixy="0.0" ixz="0.0" iyy="0.1" iyz="0.0" izz="0.1"/>
+      </inertial>
+    </link>
     <joint name="wheel_rear_right_joint" type="continuous">
       <origin rpy="-1.570796 0.000000 0.000000" xyz="0.000000 ${-wheel_base_rear} ${wheel_radius}"/>
@@ -211,3 +218,8 @@
       <limit effort="1000000.0" lower="-0.5235" upper="0.5235" velocity="100"/>
     </joint>
+    <joint name="lidar_mount_joint" type="fixed">
+      <origin rpy="0 0 0" xyz="2.2804451 0.0 0.8967377"/>
+      <parent link="base_link"/>
+      <child link="lidar_mount"/>
+    </joint>
 </robot>

File: Project/Assets/robotec_freezed_urdf_chasis/kraken_manipulator.xacro (robot description, xacro)
@@ -41,5 +41,5 @@
         <origin rpy="0 0 0" xyz="0.0 0.0 0.0"/>
         <mass value="25.0"/>
-        <inertia ixx="0.002" ixy="0.0" ixz="0.0" iyy="0.068" iyz="0.0" izz="0.067"/>
+        <inertia ixx="0.5" ixy="0.0" ixz="0.0" iyy="8.0" iyz="0.0" izz="8.0"/>
       </inertial>
       <visual>
@@ -50,5 +50,5 @@
       </visual>
       <collision>
-        <origin rpy="-0.000 -0.000000 0.000000" xyz="0.000000 0.062564 -0.000045"/>
+        <origin rpy="-0.000 -0.000000 0.000000" xyz="0.2732149 0.062564 -0.000045"/>
         <geometry>
            <box size="2.019587 0.172379 0.067739"/>
@@ -130,4 +130,49 @@
          </geometry>
        </collision>
+    </link>
+    <link name="Effector">
+      <inertial>
+        <origin rpy="0 0 0" xyz="0.0 0.0 0.0"/>
+        <mass value="1.0"/>
+        <inertia ixx="0.1" ixy="0.0" ixz="0.0" iyy="0.1" iyz="0.0" izz="0.1"/>
+      </inertial>
+      <collision>
+        <origin rpy="0 0 0" xyz="0.0 0.0 0"/>
+        <geometry>
+          <sphere  radius="0.05"/>
+        </geometry>
+      </collision>
+      <visual>
+        <origin rpy="0 0 0" xyz="0.0 0.0 0"/>
+        <geometry>
+          <box  size="0.12 0.12 0.12"/>
+        </geometry>
+      </visual>
+    </link>
+    <link name="Rest">
+      <inertial>
+        <origin rpy="0 0 0" xyz="0.0 0.0 0.0"/>
+        <mass value="10.0"/>
+        <inertia ixx="0.5" ixy="0.0" ixz="0.0" iyy="0.5" iyz="0.0" izz="0.2"/>
+      </inertial>
+      <visual>
+        <origin rpy="0 0 0" xyz="0.0 0.0 0"/>
+        <geometry>
+          <sphere  radius="0.1"/>
+        </geometry>
+      </visual>
+    </link>
+    <link name="Reach">
+      <inertial>
+        <origin rpy="0 0 0" xyz="0.0 0.0 0.0"/>
+        <mass value="10.0"/>
+        <inertia ixx="0.5" ixy="0.0" ixz="0.0" iyy="0.5" iyz="0.0" izz="0.2"/>
+      </inertial>
+      <collision>
+        <origin rpy="0 0 0" xyz="0.0 0.0 0"/>
+        <geometry>
+          <box size="1.8 0.75 1.8"/>
+        </geometry>
+      </collision>
     </link>
     <joint name="kraken_manipulator_joint_0" type="fixed">
@@ -172,3 +217,18 @@
       <limit effort="1000.0" lower="0" upper="0.3" velocity="1.0"/>
     </joint>
+    <joint name="rest_joint" type="fixed">
+      <origin rpy="0 0 0" xyz="${manip_x+0.2558164} -1.2641881 1.6814755"/>
+      <parent link="base_link"/>
+      <child link="Rest"/>
+    </joint>
+    <joint name="reach_joint" type="fixed">
+      <origin rpy="-0.10471975512 0 0" xyz="${manip_x-0.4} -1.65 1.6"/>
+      <parent link="base_link"/>
+      <child link="Reach"/>
+    </joint>
+    <joint name="effector_joint" type="fixed">
+      <origin rpy="0 0 0" xyz="-0.0100173 -0.0020601 0.4332509"/>
+      <parent link="kraken_manipulator_link_4"/>
+      <child link="Effector"/>
+    </joint>
 </robot>

Commit message: Added conveyor belt
Signed-off-by: Paweł Budziszewski <pawel.budziszewski@robotec.ai>

File: Project/Assets/robotec_freezed_urdf_chasis/kraken_chasis.xacro (robot description, xacro)
@@ -174,4 +174,17 @@
       </inertial>
     </link>
+    <link name="conveyor_belt">
+      <inertial>
+        <origin rpy="0 0 0" xyz="0 0 0"/>
+        <mass value="5.0"/>
+        <inertia ixx="0.1" ixy="0.0" ixz="0.0" iyy="0.5" iyz="0.0" izz="0.5"/>
+      </inertial>
+      <visual>
+        <origin rpy="0 0 0" xyz="0 0 0"/>
+        <geometry>
+          <mesh filename="meshes/ConveyorBelt/ConveyorBelt.dae" scale="1.0 1.0 1.0"/>
+        </geometry>
+      </visual>
+    </link>
     <joint name="wheel_rear_right_joint" type="continuous">
       <origin rpy="-1.570796 0.000000 0.000000" xyz="0.000000 ${-wheel_base_rear} ${wheel_radius}"/>
@@ -223,3 +236,8 @@
       <child link="lidar_mount"/>
     </joint>
+    <joint name="conveyor_belt_joint" type="fixed">
+      <origin rpy="0 0 1.571" xyz="1.1043353 0 0.0"/>
+      <parent link="base_link"/>
+      <child link="conveyor_belt"/>
+    </joint>
 </robot>
