Commit message: Added description of manipulator part + fixes in xacro and descroption
Signed-off-by: Paweł Budziszewski <pawel.budziszewski@robotec.ai>

File: Project/Assets/robotec_freezed_urdf_chasis/kraken_manipulator.xacro (robot description, xacro)
@@ -150,4 +150,11 @@
       </visual>
     </link>
+    <link name="RetrievalChute">
+      <inertial>
+        <origin rpy="0 0 0" xyz="0.0 0.0 0.0"/>
+        <mass value="1.0"/>
+        <inertia ixx="0.1" ixy="0.0" ixz="0.0" iyy="0.1" iyz="0.0" izz="0.1"/>
+      </inertial>
+    </link>
     <link name="Rest">
       <inertial>
@@ -169,10 +176,10 @@
         <inertia ixx="0.5" ixy="0.0" ixz="0.0" iyy="0.5" iyz="0.0" izz="0.2"/>
       </inertial>
-      <collision>
+      <visual>
         <origin rpy="0 0 0" xyz="0.0 0.0 0"/>
         <geometry>
           <box size="1.8 0.75 1.8"/>
         </geometry>
-      </collision>
+      </visual>
     </link>
     <joint name="kraken_manipulator_joint_0" type="fixed">
@@ -232,3 +239,8 @@
       <child link="Effector"/>
     </joint>
+    <joint name="retrieval_chute_joint" type="fixed">
+      <origin rpy="0 0 0" xyz="1.3339844 -0.2378311 1.3847573"/>
+      <parent link="base_link"/>
+      <child link="RetrievalChute"/>
+    </joint>
 </robot>
