Commit message: Fixed Effector rotation
Incorrect rotation of the Effector object caused the manipulator was not abble to reach apples while pickong

Signed-off-by: Paweł Budziszewski <pawel.budziszewski@robotec.ai>

File: Project/Assets/applekraken_urdf/apple_kraken.xacro (robot description, xacro)
@@ -443,5 +443,5 @@
     </joint>
     <joint name="effector_joint" type="fixed">
-      <origin rpy="0 0 0" xyz="-0.0100173 -0.0020601 0.4332509"/>
+      <origin rpy="1.571 0 1.571" xyz="-0.0100173 -0.0020601 0.4332509"/>
       <parent link="kraken_manipulator_link_4"/>
       <child link="Effector"/>
